Commit message: feat: implement system manager and teleop nodes, add web-based GUI, and update robot configuration and maps

File: Group 6 TITAN: Trash Interception and Termination Autonomous Navigator/titan_ws/src/titan_description/urdf/robot_core.xacro (robot description, xacro)
@@ -42,4 +42,10 @@
         </xacro:inertial_box>
     </link>
+    <joint name="imu_joint" type="fixed">
+        <parent link="chassis"/>
+        <child link="imu_link"/>
+        <origin xyz="0 0 -0.01" rpy="${pi} 0 0"/>
+    </joint>
+    <link name="imu_link"></link>
     <xacro:macro name="wheel" params="prefix x_reflect y_reflect">
         <joint name="${prefix}_wheel_joint" type="continuous">
